Commit message: Add TCP links and update tip links for Yumi robot's left and right arms

File: yumi_description/urdf/yumi.xacro (robot description, xacro)
@@ -254,4 +254,10 @@
       </collision>
     </link>
+    <link name="yumi_tcp_r"/>
+    <joint name="yumi_tcp_r_joint" type="fixed">
+      <parent link="yumi_link_7_r"/>
+      <child link="yumi_tcp_r"/>
+      <origin xyz="0 0 0.138" rpy="0 0 0"/>
+    </joint>
     <!--///////////////////////////////////// LEFT ARM ////////////////////////////////  -->
     <!-- joint between body and link_1_l -->
@@ -472,4 +478,10 @@
       </collision>
     </link>
+    <link name="yumi_tcp_l"/>
+    <joint name="yumi_tcp_l_joint" type="fixed">
+      <parent link="yumi_link_7_l"/>
+      <child link="yumi_tcp_l"/>
+      <origin xyz="0 0 0.138" rpy="0 0 0"/>
+    </joint>
     <!--Extensions -->
     <xacro:yumi_gazebo name="${name}" />
